File: Hardware/Sumo-Michi-Go.kicad_sch (KiCad schematic)
At the start: 14 parts, among them J1 ENTRADA, J2 PUENTE_H, J3 Conn_01x09_Pin, J4 SENSOR_INFRAROJO_1, J5 ULTRASONIDO_1, J6 ULTRASONIDO_2, J7 SENSOR_INFRAROJO_2, J8 SENSOR_INFRAROJO_3, SW1 SWITCH_ON_OFF, SW2 SW_DE_INICIO_ROBOT, U2 LM7805_TO220

Commit message: esta es la ultima
Parts:
- removed U2: LM7805_TO220, Package_TO_SOT_THT:TO-220-3_Vertical, symbol Regulator_Linear:LM7805_TO220
- added J10: SALIDA_STEPDOWN, TerminalBlock:TerminalBlock_Altech_AK300-2_P5.00mm, symbol Connector:Screw_Terminal_01x02
- added J9: ENTRADA_STEPDOWN, TerminalBlock:TerminalBlock_Altech_AK300-2_P5.00mm, symbol Connector:Screw_Terminal_01x02
- SW1: footprint Button_Switch_THT:SW_DIP_SPSTx01_Slide_9.78x4.72mm_W7.62mm_P2.54mm -> llave depalanca:SW_100SP1T1B1M1QEH
Connections:
- net +5V: now also J10.1 (Pin_1)
- net GND: now also J10.2 (Pin_2), J9.1 (Pin_1)
- net entrada del step down: now reaches D1.2 (A), R1.2
- net entrada del step down: now also J9.2 (Pin_2)
