File: Hardware/Sumo-Michi-Go.kicad_sch (KiCad schematic)
At the start: 14 parts, among them J1 ENTRADA, J2 PUENTE_H, J3 Conn_01x09_Pin, J4 SENSOR_INFRAROJO_1, J5 ULTRASONIDO_1, J6 ULTRASONIDO_2, J7 SENSOR_INFRAROJO_2, J8 SENSOR_INFRAROJO_3, SW1 SWITCH_ON_OFF, SW2 SW_DE_INICIO_ROBOT, U2 LM7805_TO220

Commit message: esta cae
Parts:
- removed U2: LM7805_TO220, Package_TO_SOT_THT:TO-220-3_Vertical, symbol Regulator_Linear:LM7805_TO220
- added J10, J9: ENTRADA, TerminalBlock:TerminalBlock_Altech_AK300-2_P5.00mm, symbol Connector:Screw_Terminal_01x02
- SW1: footprint Button_Switch_THT:SW_DIP_SPSTx01_Slide_9.78x4.72mm_W7.62mm_P2.54mm -> llave depalanca:SW_100SP1T1B1M1QEH
Connections:
- net +5V: now also J10.1 (Pin_1)
- net GND: now also J10.2 (Pin_2), J9.1 (Pin_1)
- net ENTRADA_STEPDOWN: now reaches D1.2 (A), R1.2
- net ENTRADA_STEPDOWN: now also J9.2 (Pin_2)

Commit message: ultima
Parts:
- removed J2: PUENTE_H, Connector_PinSocket_2.54mm:PinSocket_1x08_P2.54mm_Vertical, symbol Connector:Conn_01x08_Pin
- added J11: Conn_01x10, Connector_PinHeader_2.54mm:PinHeader_1x10_P2.54mm_Vertical, symbol Connector_Generic:Conn_01x10
- added J2: Conn_01x04, Connector_PinHeader_2.54mm:PinHeader_1x04_P2.54mm_Vertical, symbol Connector_Generic:Conn_01x04
- added R2: R, Resistor_SMD:R_0805_2012Metric, symbol Device:R
Connections:
- net L_IS  is gone; now on net PWM2: A1.6 (D3)
- net +5V: now also J5.3 (Pin_3), J6.3 (Pin_3), J11.7 (Pin_7), J11.9 (Pin_9), R2.1; no longer J5.1 (Pin_1), J6.1 (Pin_1)
- net 5v_arduino: now also J3.7 (Pin_7), J3.8 (Pin_8), J3.9 (Pin_9), J2.2 (Pin_2); no longer J3.4 (Pin_4), J3.5 (Pin_5), J3.6 (Pin_6)
- net ENABLE 1: now also J11.4 (Pin_4)
- net ENABLE 2: now also J11.6 (Pin_6)
- net GND: now also J11.10 (Pin_10), J11.5 (Pin_5), J2.1 (Pin_1)
- net PWM 1: now also A1.14 (D11), J11.1 (Pin_1); no longer A1.8 (D5)
- net PWM2: now also J11.8 (Pin_8); no longer A1.9 (D6)
- net eccho 1: now also A1.23 (A4); no longer A1.22 (A3)
- net sensor 1: now also A1.21 (A2), J3.5 (Pin_5); no longer A1.13 (D10), J3.8 (Pin_8)
- net sensor 2: now also A1.20 (A1), J3.4 (Pin_4); no longer A1.14 (D11), J3.9 (Pin_9)
- net sensor 3: now also A1.22 (A3), J3.6 (Pin_6); no longer A1.12 (D9), J3.7 (Pin_7)
- net sensor_distancia1: now also A1.24 (A5); no longer A1.23 (A4)
- net sensor_distancia2: now also A1.25 (A6); no longer A1.24 (A5)
- net sensor_distancia3: now also A1.26 (A7); no longer A1.25 (A6)
- net trig 1: now also A1.15 (D12), J5.1 (Pin_1); no longer A1.21 (A2), J5.3 (Pin_3)
- net trig 2: now also A1.9 (D6), J6.1 (Pin_1); no longer A1.20 (A1), J6.3 (Pin_3)
- net at SW2.2 (B): now also A1.5 (D2), R2.2; no longer A1.15 (D12)
- net R_IS  renamed display
- net display: now also J2.4 (Pin_4)
- new net PWM 3: A1.13 (D10), J11.2 (Pin_2)
- new net PWM 4: A1.12 (D9), J11.3 (Pin_3)
- new net display 2: A1.8 (D5), J2.3 (Pin_3)
Other:
- moved on the sheet: SW2

Commit message: PCB nuevo
Parts:
- removed J11: Conn_01x10, Connector_PinHeader_2.54mm:PinHeader_1x10_P2.54mm_Vertical, symbol Connector_Generic:Conn_01x10
- removed J2: Conn_01x04, Connector_PinHeader_2.54mm:PinHeader_1x04_P2.54mm_Vertical, symbol Connector_Generic:Conn_01x04
- added D2, D3: LED, LED_THT:LED_D5.0mm_Clear, symbol Device:LED
- added J11: PUENTEH_A, TerminalBlock:TerminalBlock_Altech_AK300-2_P5.00mm, symbol Connector:Screw_Terminal_01x02
- added J12: PUENTEH_B, TerminalBlock:TerminalBlock_Altech_AK300-2_P5.00mm, symbol Connector:Screw_Terminal_01x02
- added J13: PUENTEH_A, Connector_PinSocket_2.54mm:PinSocket_1x05_P2.54mm_Vertical, symbol Connector:Conn_01x05_Pin
- added J14: PUENTEH_B, Connector_PinSocket_2.54mm:PinSocket_1x05_P2.54mm_Vertical, symbol Connector:Conn_01x05_Pin
- added R3, R4: R, Resistor_SMD:R_0805_2012Metric, symbol Device:R
- D1: footprint Inductor_SMD:L_0805_2012Metric_Pad1.15x1.40mm_HandSolder -> LED_THT:LED_D5.0mm_Clear
- J3: value Conn_01x09_Pin -> Sensores_de_piso
Connections:
- net +5V: now also J13.1 (Pin_1), J14.1 (Pin_1)
- net GND: now also D2.1 (K), D3.1 (K), J11.1 (Pin_1), J12.1 (Pin_1), J13.5 (Pin_5), J14.5 (Pin_5)
- net VCC: now also J11.2 (Pin_2), J12.2 (Pin_2)
- net SW_DE_INICIO: now reaches A1.5 (D2), R2.2, SW2.2 (B)
- net ENABLE 1 renamed ENABLE_B
- net ENABLE_B: now also J14.4 (Pin_4)
- net ENABLE 2 renamed ENABLE_A
- net ENABLE_A: now also J13.4 (Pin_4)
- net PWM 1 renamed PWM2_A
- net PWM2_A: now also J13.3 (Pin_3)
- net PWM 3 renamed PWM1_B
- net PWM1_B: now also J14.2 (Pin_2)
- net PWM 4 renamed PWM2_B
- net PWM2_B: now also J14.3 (Pin_3)
- net PWM2 renamed PWM1_A
- net PWM1_A: now also J13.2 (Pin_2)
- net display renamed LED_A
- net LED_A: now also R3.2
- net display 2 renamed LED_B
- net LED_B: now also R4.2
- new net: D2.2 (A), R3.1
- new net: D3.2 (A), R4.1
Other:
- moved on the sheet: A1, D1, J1, J10, J3, J4, J5, J6, J7, J8, J9, R1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
