File: Hardware/Sumo-Michi-Go.kicad_pcb (KiCad board)
At the start: 2 copper layers, 84.3 x 69.6 mm, 14 parts, among them J1 ENTRADA, J2 PUENTE_H, J3 Conn_01x09_Pin, J4 SENSOR_INFRAROJO_1, J5 ULTRASONIDO_1, J6 ULTRASONIDO_2, J7 SENSOR_INFRAROJO_2, J8 SENSOR_INFRAROJO_3, SW1 SWITCH_ON_OFF, SW2 SW_DE_INICIO_ROBOT, U2 LM7805_TO220

Commit message: esta es la ultima
Parts:
- removed U2: LM7805_TO220, Package_TO_SOT_THT:TO-220-3_Vertical
- added J10: ENTRADA, TerminalBlock:TerminalBlock_Altech_AK300-2_P5.00mm, F.Cu at (24.3, 34.8)
- added J9: ENTRADA, TerminalBlock:TerminalBlock_Altech_AK300-2_P5.00mm, F.Cu at (24.3, 46.6)
- SW1: footprint Button_Switch_THT:SW_DIP_SPSTx01_Slide_9.78x4.72mm_W7.62mm_P2.54mm -> llave depalanca:SW_100SP1T1B1M1QEH
- moved SW1 0.32 mm to (29.8, 65.3)
Connections:
- net Net-(D1-A) renamed entrada del step down
Routing:
- net +5V: track 95.6 -> 88.3 mm
- net entrada del step down: track 11.9 -> 8.75 mm
- net VCC: track 64.8 -> 62.6 mm

Commit message: esta_cae
Parts:
- moved J9 4.15 mm to (24.3, 42.5)
- moved R1 3.29 mm to (24.1, 57.1), turned to 90 degrees
- moved D1 2.68 mm to (25.1, 54.0)
- moved J10 0.60 mm to (24.4, 35.4), turned to 90 degrees
- moved SW1 0.32 mm to (29.8, 65.0)
Connections:
- net entrada del step down renamed entrada_stepdown
Routing:
- net VCC: track 62.6 -> 71.6 mm
- net Net-(J1-Pin_2): track 15.7 -> 19.3 mm
- net +5V: track 88.3 -> 86.9 mm

Commit message: esta cae
Parts:
- moved J10 9.27 mm to (24.1, 26.1), turned to -90 degrees
- moved D1 2.28 mm to (23.2, 52.7), turned to 0 degrees
- moved J9 1.27 mm to (24.3, 41.2)
- moved R1 0.20 mm to (24.3, 57.1)
Connections:
- net entrada_stepdown renamed ENTRADA_STEPDOWN
Routing:
- net VCC: track 71.6 -> 80.5 mm
- net ENTRADA_STEPDOWN: track 8.79 -> 10.1 mm
- net +5V: track 86.9 -> 85.7 mm

Commit message: ultima
Parts:
- added J11: Conn_01x10, Connector_PinHeader_2.54mm:PinHeader_1x10_P2.54mm_Vertical, F.Cu at (89.2, 76.2)
- added R2: R, Resistor_SMD:R_0805_2012Metric, F.Cu at (49.1, 62.4)
- J2: value PUENTE_H -> Conn_01x04; footprint Connector_PinSocket_2.54mm:PinSocket_1x08_P2.54mm_Vertical -> Connector_PinHeader_2.54mm:PinHeader_1x04_P2.54mm_Vertical
- moved J3 55.4 mm to (90.6, 24.4), turned to 0 degrees
- moved SW2 19.2 mm to (48.8, 71.7), turned to -90 degrees
- moved J6 16.4 mm to (75.7, 23.7)
- moved J2 14.5 mm to (38.1, 66.4), turned to 180 degrees
- moved SW1 11.9 mm to (20.6, 72.7), turned to 90 degrees
- moved J5 2.97 mm to (62.3, 23.7), turned to 0 degrees
- moved R1 1.42 mm to (23.1, 58.0), turned to 180 degrees
Connections:
- net R_IS  renamed display
- A1 pad 12: sensor 3 -> PWM 4
- A1 pad 13: sensor 1 -> PWM 3
- A1 pad 14: sensor 2 -> PWM 1
- A1 pad 15: Net-(A1-D12) -> trig 1
- A1 pad 20: trig 2 -> sensor 2
- A1 pad 21: trig 1 -> sensor 1
- A1 pad 22: eccho 1 -> sensor 3
- A1 pad 23: sensor_distancia1 -> eccho 1
- A1 pad 24: sensor_distancia2 -> sensor_distancia1
- A1 pad 25: sensor_distancia3 -> sensor_distancia2
- A1 pad 26: unconnected-(A1-A7-Pad26) -> sensor_distancia3
- A1 pad 5: unconnected-(A1-D2-Pad5) -> Net-(A1-D2)
- A1 pad 6: L_IS  -> PWM2
- A1 pad 8: PWM 1 -> display 2
- A1 pad 9: PWM2 -> trig 2
- J2 pad 1: VCC -> GND
- J2 pad 2: GND -> 5v_arduino
- J2 pad 3: L_IS  -> display 2
- J3 pad 4: 5v_arduino -> sensor 2
- J3 pad 5: 5v_arduino -> sensor 1
- J3 pad 6: 5v_arduino -> sensor 3
- J3 pad 7: sensor 3 -> 5v_arduino
- J3 pad 8: sensor 1 -> 5v_arduino
- J3 pad 9: sensor 2 -> 5v_arduino
- J5 pad 1: +5V -> trig 1
- J5 pad 3: trig 1 -> +5V
- J6 pad 1: +5V -> trig 2
- J6 pad 3: trig 2 -> +5V
- SW2 pad 2: Net-(A1-D12) -> Net-(A1-D2)
Routing:
- net +5V: track 85.7 -> 229.5 mm
- net trig 1: track 14.5 -> 86.7 mm
- net display 2: track 0.00 -> 47.5 mm
- net trig 2: track 35.3 -> 82.0 mm
- net PWM 4: track 0.00 -> 35.0 mm
- net VCC: track 80.5 -> 45.9 mm
- net PWM 3: track 0.00 -> 34.2 mm
- net Net-(A1-D2): track 0.00 -> 29.0 mm
- net L_IS : track 25.8 -> 0.00 mm
- net GND: track 0.00 -> 22.9 mm, vias 0 -> 2
- net eccho 2: track 31.4 -> 15.5 mm
- net Net-(A1-D12): track 15.4 -> 0.00 mm
- net sensor 3: track 54.7 -> 41.4 mm
- net 5v_arduino: track 89.1 -> 100.6 mm
- net display: track 25.8 -> 36.0 mm
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Other:
- board size 84.3 x 69.6 mm -> 87.6 x 69.6 mm

Commit message: basta porfavor
Parts:
- moved R1 2.05 mm to (24.3, 59.7), turned to 90 degrees
Routing:
- net VCC: track 45.9 -> 62.2 mm
- net ENTRADA_STEPDOWN: track 10.1 -> 12.6 mm
Changed lines of the file:
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@@
 	(footprint "Resistor_SMD:R_0805_2012Metric"
 		(layer "B.Cu")
-		(at 23.1075 57.97 180)
+		(at 24.265 59.66 90)
 		(descr "Resistor SMD 0805 (2012 Metric), square (rectangular) end terminal, IPC_7351 nominal, (Body size source: IPC-SM-782 page 72, https://www.pcb-3d.com/wordpress/wp-content/uploads/ipc-sm-782a_amendment_1_and_2.pdf), generated with kicad-footprint-generator")
 		(tags "resistor")
 		(property "Reference" "R1"
-			(at 0 1.65 0)
+			(at 0 1.65 90)
 			(layer "B.SilkS")
 			(hide yes)
@@
 		)
 		(property "Value" "R"
-			(at -0.0875 -2.5 0)
+			(at -0.0875 -2.5 90)
 			(layer "B.Fab")
 			(effects
@@
 		)
 		(property "Datasheet" ""
-			(at 0 0 0)
+			(at 0 0 270)
 			(unlocked yes)
 			(layer "B.Fab")
@@
 		)
 		(property "Description" "Resistor"
-			(at 0 0 0)
+			(at 0 0 270)
 			(unlocked yes)
 			(layer "B.Fab")
@@
 		(attr smd)
 		(fp_line
+			(start -0.227064 -0.735)
+			(end 0.227064 -0.735)
+			(stroke
+				(width 0.12)
+				(type solid)
+			)
+			(layer "B.SilkS")
+		)
+		(fp_line
 			(start -0.227064 0.735)
 			(end 0.227064 0.735)
@@
 		)
 		(fp_line
-			(start -0.227064 -0.735)
-			(end 0.227064 -0.735)
-			(stroke
-				(width 0.12)
-				(type solid)
-			)
-			(layer "B.SilkS")
+			(start 1.68 -0.95)
+			(end -1.68 -0.95)
+			(stroke
+				(width 0.05)
+				(type solid)
+			)
+			(layer "B.CrtYd")
+		)
+		(fp_line
+			(start -1.68 -0.95)
+			(end -1.68 0.95)
+			(stroke
+				(width 0.05)
+				(type solid)
+			)
+			(layer "B.CrtYd")
 		)
 		(fp_line
@@
 		)
 		(fp_line
-			(start 1.68 -0.95)
-			(end -1.68 -0.95)
-			(stroke
-				(width 0.05)
-				(type solid)
-			)
-			(layer "B.CrtYd")
-		)
-		(fp_line
 			(start -1.68 0.95)
 			(end 1.68 0.95)
@@
 		)
 		(fp_line
-			(start -1.68 -0.95)
-			(end -1.68 0.95)
-			(stroke
-				(width 0.05)
-				(type solid)
-			)
-			(layer "B.CrtYd")
+			(start 1 -0.625)
+			(end -1 -0.625)
+			(stroke
+				(width 0.1)
+				(type solid)
+			)
+			(layer "B.Fab")
+		)
+		(fp_line
+			(start -1 -0.625)
+			(end -1 0.625)
+			(stroke
+				(width 0.1)
+				(type solid)
+			)
+			(layer "B.Fab")
 		)
 		(fp_line
@@
 		)
 		(fp_line
-			(start 1 -0.625)
-			(end -1 -0.625)
-			(stroke
-				(width 0.1)
-				(type solid)
-			)
-			(layer "B.Fab")
-		)
-		(fp_line
 			(start -1 0.625)
 			(end 1 0.625)
@@
 			(layer "B.Fab")
 		)
-		(fp_line
-			(start -1 -0.625)
-			(end -1 0.625)
-			(stroke
-				(width 0.1)
-				(type solid)
-			)
-			(layer "B.Fab")
-		)
 		(fp_text user "${REFERENCE}"
-			(at 0 0 0)
+			(at 0 0 90)
 			(layer "B.Fab")
 			(effects
@@
 		)
 		(pad "1" smd roundrect
-			(at -0.9125 0 180)
+			(at -0.9125 0 90)
 			(size 1.025 1.4)
 			(layers "B.Cu" "B.Mask" "B.Paste")
@@
 		)
 		(pad "2" smd roundrect
-			(at 0.9125 0 180)
+			(at 0.9125 0 90)
 			(size 1.025 1.4)
 			(layers "B.Cu" "B.Mask" "B.Paste")
@@
 	)
 	(gr_text "que significa \n{dblquote}bro respeta{dblquote}?\n"
-		(at -7.21 57.94 270)
+		(at 93.56 71.73 270)
 		(layer "B.Cu")
 		(effects
@@
 	)
 	(segment
+		(start 25.42 66.14)
+		(end 25.42 70.94)
+		(width 1.5)
+		(layer "B.Cu")
+		(net 6)
+	)
+	(segment
 		(start 28.56 63.78)
 		(end 28.56 44.27)
@@
 	)
 	(segment
+		(start 25.42 70.94)
+		(end 23.693 72.667)
+		(width 1.5)
+		(layer "B.Cu")
+		(net 6)
+	)
+	(segment
+		(start 23.693 72.667)
+		(end 20.6425 72.667)
+		(width 1.5)
+		(layer "B.Cu")
+		(net 6)
+	)
+	(segment
 		(start 34.688 38.142)
 		(end 37.312 38.142)
@@
 	)
 	(segment
+		(start 24.265 60.5725)
+		(end 24.265 64.985)
+		(width 1.5)
+		(layer "B.Cu")
+		(net 6)
+	)
+	(segment
+		(start 24.265 64.985)
+		(end 25.42 66.14)
+		(width 1.5)
+		(layer "B.Cu")
+		(net 6)
+	)
+	(segment
 		(start 20.6425 72.667)
 		(end 25.663 72.667)
@@
 	)
 	(segment
-		(start 24.265 56.2375)
-		(end 24.265 52.72)
-		(width 1.5)
-		(layer "B.Cu")
-		(net 28)
-	)
-	(segment
 		(start 24.265 46.18)
 		(end 24.265 52.72)
 		(width 1.5)
 		(layer "B.Cu")
+		(net 28)
+	)
+	(segment
+		(start 24.265 52.72)
+		(end 24.265 58.7475)
+		(width 1.5)
+		(layer "B.Cu")

Commit message: PCB nuevo
Parts:
- removed J2: Conn_01x04, Connector_PinHeader_2.54mm:PinHeader_1x04_P2.54mm_Vertical
- added D2: LED, LED_THT:LED_D5.0mm_Clear, F.Cu at (42.6, 67.1)
- added D3: LED, LED_THT:LED_D5.0mm_Clear, F.Cu at (35.9, 67.1)
- added J12: PUENTEH_B, TerminalBlock:TerminalBlock_Altech_AK300-2_P5.00mm, F.Cu at (54.5, 87.8)
- added J13: PUENTEH_A, Connector_PinSocket_2.54mm:PinSocket_1x05_P2.54mm_Vertical, F.Cu at (61.0, 84.2)
- added J14: PUENTEH_B, Connector_PinSocket_2.54mm:PinSocket_1x05_P2.54mm_Vertical, F.Cu at (85.5, 84.3)
- added R3: R, Resistor_SMD:R_0805_2012Metric, F.Cu at (42.6, 60.0)
- added R4: R, Resistor_SMD:R_0805_2012Metric, F.Cu at (35.9, 60.0)
- D1: footprint Inductor_SMD:L_0805_2012Metric_Pad1.15x1.40mm_HandSolder -> LED_THT:LED_D5.0mm_Clear
- J11: value Conn_01x10 -> PUENTEH_A; footprint Connector_PinHeader_2.54mm:PinHeader_1x10_P2.54mm_Vertical -> TerminalBlock:TerminalBlock_Altech_AK300-2_P5.00mm
- J3: value Conn_01x09_Pin -> Sensores_de_piso
- moved J11 48.6 mm to (42.0, 87.8), turned to 180 degrees
- moved J1 17.3 mm to (25.6, 87.8), turned to 180 degrees
- moved SW2 6.50 mm to (47.5, 78.1), turned to 180 degrees
- moved SW1 4.88 mm to (25.3, 74.0), turned to 0 degrees
- moved D1 1.83 mm to (21.7, 53.8)
- moved R2 0.71 mm to (48.4, 62.4)
Connections:
- net Net-(A1-D2) renamed SW_DE_INICIO
- A1 pad 10: ENABLE 2 -> ENABLE_A
- A1 pad 11: ENABLE 1 -> ENABLE_B
- A1 pad 12: PWM 4 -> PWM2_B
- A1 pad 13: PWM 3 -> PWM1_B
- A1 pad 14: PWM 1 -> PWM2_A
- A1 pad 6: PWM2 -> PWM1_A
- A1 pad 7: display -> LED_A
- A1 pad 8: display 2 -> LED_B
- J11 pad 1: PWM 1 -> GND
- J11 pad 2: PWM 3 -> VCC
Routing:
- net PWM2_A: track 0.00 -> 70.2 mm
- net display 2: track 47.5 -> 0.00 mm
- net 5v_arduino: track 100.6 -> 58.5 mm
- net LED_B: track 0.00 -> 39.0 mm
- net PWM2_B: track 0.00 -> 37.2 mm
- net PWM1_B: track 0.00 -> 37.2 mm
- net ENABLE_B: track 0.00 -> 37.2 mm
- net LED_A: track 0.00 -> 37.2 mm
- net PWM1_A: track 0.00 -> 36.4 mm
- net display: track 36.0 -> 0.00 mm
- net PWM2: track 35.1 -> 0.00 mm
- net PWM 4: track 35.0 -> 0.00 mm
- net ENABLE 1: track 35.0 -> 0.00 mm
- net ENABLE_A: track 0.00 -> 34.3 mm
- net PWM 3: track 34.2 -> 0.00 mm
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Other:
- board size 87.6 x 69.6 mm -> 87.4 x 80.7 mm
